File: Electronics/Peltier Driver/_autosave-PID_electronics.kicad_sch (KiCad schematic)
At the start: 15 parts, among them J1 Conn_01x05, J2 Conn_01x03, Q3 2N7000, U1 LF412

Commit message: Board revision
Parts:
- R3: footprint Resistor_THT:R_Axial_DIN0207_L6.3mm_D2.5mm_P15.24mm_Horizontal -> Resistor_THT:R_Axial_DIN0207_L6.3mm_D2.5mm_P10.16mm_Horizontal
Changed lines of the file:
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@@
     (property "Reference" "R3" (id 0) (at 76.2 63.5 90))
     (property "Value" "10K" (id 1) (at 76.2 66.04 90))
-    (property "Footprint" "Resistor_THT:R_Axial_DIN0207_L6.3mm_D2.5mm_P15.24mm_Horizontal" (id 2) (at 76.2 62.738 90)
+    (property "Footprint" "Resistor_THT:R_Axial_DIN0207_L6.3mm_D2.5mm_P10.16mm_Horizontal" (id 2) (at 76.2 62.738 90)
       (effects (font (size 1.27 1.27)) hide)
     )
@@
     )
     (path "/f3c271ed-c988-4d5a-9710-8799a0d2f035"
-      (reference "R3") (unit 1) (value "10K") (footprint "Resistor_THT:R_Axial_DIN0207_L6.3mm_D2.5mm_P15.24mm_Horizontal")
+      (reference "R3") (unit 1) (value "10K") (footprint "Resistor_THT:R_Axial_DIN0207_L6.3mm_D2.5mm_P10.16mm_Horizontal")
     )
     (path "/a226fb1b-5df9-4dca-9160-13ce52ad4833"
