File: Electronics/Peltier Driver/PID_electronics.kicad_sch (KiCad schematic)
At the start: 15 parts, among them J1 Conn_01x05, J2 Conn_01x03, Q3 2N7000, U1 LF412

Commit message: Added Bulk decoupling capacitors and optional snubber network
Parts:
- added C4, C5: 1000 uF, Capacitor_THT:CP_Radial_D10.0mm_P5.00mm, symbol Device:C_Polarized_Small
- added C6: C_Small, Capacitor_THT:CP_Radial_D10.0mm_P5.00mm, symbol Device:C_Small
- added R10: R, Resistor_THT:R_Axial_DIN0207_L6.3mm_D2.5mm_P10.16mm_Horizontal, symbol Device:R
- C1: value 10 nF -> 1 nF
- R3: footprint Resistor_THT:R_Axial_DIN0207_L6.3mm_D2.5mm_P15.24mm_Horizontal -> Resistor_THT:R_Axial_DIN0207_L6.3mm_D2.5mm_P10.16mm_Horizontal
Connections:
- net +15V: now also C5.1
- net -15V: now also C4.2
- net GNDREF: now also C4.1, C5.2, C6.2
- net at J2.1 (Pin_1), R7.2: now also R10.1
- new net: C6.1, R10.2
Other:
- moved on the sheet: R8
