File: Electronics/Peltier Driver/PID_electronics.kicad_sch (KiCad schematic)
At the start: 21 parts, among them J1 Conn_01x05, J2 Conn_01x03, Q3 2N7000, U1 LF412

Commit message: Replaced Opamp footprint with socket footprint
Parts:
- U1: footprint Package_DIP:DIP-8_W10.16mm_LongPads -> Package_DIP:DIP-8_W7.62mm_Socket_LongPads
- renumbered C6 to C7, C7 to C8
Changed lines of the file:
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@@
   (symbol (lib_id "Device:C_Small") (at 163.83 60.96 0) (mirror y) (unit 1)
     (in_bom yes) (on_board yes)
-    (property "Reference" "C6" (id 0) (at 160.02 60.96 0)
+    (property "Reference" "C7" (id 0) (at 160.02 60.96 0)
       (effects (font (size 0.8 0.8)) (justify right))
     )
@@
     (property "Reference" "U1" (id 0) (at 144.145 64.77 0))
     (property "Value" "LF412" (id 1) (at 144.145 62.23 0))
-    (property "Footprint" "Package_DIP:DIP-8_W10.16mm_LongPads" (id 2) (at 151.765 72.39 0)
+    (property "Footprint" "Package_DIP:DIP-8_W7.62mm_Socket_LongPads" (id 2) (at 151.765 72.39 0)
       (effects (font (size 1.27 1.27)) hide)
     )
@@
       (effects (font (size 1.27 1.27)) (justify left) hide)
     )
-    (property "Footprint" "Package_DIP:DIP-8_W10.16mm_LongPads" (id 2) (at 153.035 72.39 0)
+    (property "Footprint" "Package_DIP:DIP-8_W7.62mm_Socket_LongPads" (id 2) (at 153.035 72.39 0)
       (effects (font (size 1.27 1.27)) hide)
     )
@@
     (property "Reference" "U1" (id 0) (at 193.675 72.39 0))
     (property "Value" "LF412" (id 1) (at 193.675 69.85 0))
-    (property "Footprint" "Package_DIP:DIP-8_W10.16mm_LongPads" (id 2) (at 186.055 74.93 0)
+    (property "Footprint" "Package_DIP:DIP-8_W7.62mm_Socket_LongPads" (id 2) (at 186.055 74.93 0)
       (effects (font (size 1.27 1.27)) hide)
     )
@@
   (symbol (lib_id "Device:C_Small") (at 163.83 83.82 0) (unit 1)
     (in_bom yes) (on_board yes)
-    (property "Reference" "C7" (id 0) (at 160.02 83.82 0)
+    (property "Reference" "C8" (id 0) (at 160.02 83.82 0)
       (effects (font (size 0.8 0.8)) (justify left))
     )
@@
       (reference "C5") (unit 1) (value "1000 uF") (footprint "Capacitor_THT:CP_Radial_D10.0mm_P5.00mm")
     )
-    (path "/29bc48cf-d8fe-4214-b2d7-759437472a93"
-      (reference "C6") (unit 1) (value "C_Small") (footprint "Capacitor_THT:C_Axial_L3.8mm_D2.6mm_P7.50mm_Horizontal")
-    )
     (path "/8ea27319-6561-48d0-833e-434a565ff3b2"
       (reference "C6") (unit 1) (value "C_Small") (footprint "Capacitor_THT:CP_Radial_D10.0mm_P5.00mm")
     )
+    (path "/29bc48cf-d8fe-4214-b2d7-759437472a93"
+      (reference "C7") (unit 1) (value "C_Small") (footprint "Capacitor_THT:C_Axial_L3.8mm_D2.6mm_P7.50mm_Horizontal")
+    )
     (path "/dbe3ed1d-1e50-4ccd-ba3e-6e66d24024b4"
-      (reference "C7") (unit 1) (value "C_Small") (footprint "Capacitor_THT:C_Axial_L3.8mm_D2.6mm_P7.50mm_Horizontal")
+      (reference "C8") (unit 1) (value "C_Small") (footprint "Capacitor_THT:C_Axial_L3.8mm_D2.6mm_P7.50mm_Horizontal")
     )
     (path "/eecd43dc-9458-46d0-afaa-bc2f0fdbe268"
@@
     )
     (path "/2a9cad4f-2bb5-49ad-b88c-871995bf30a0"
-      (reference "U1") (unit 1) (value "LF412") (footprint "Package_DIP:DIP-8_W10.16mm_LongPads")
+      (reference "U1") (unit 1) (value "LF412") (footprint "Package_DIP:DIP-8_W7.62mm_Socket_LongPads")
     )
     (path "/532cb9ef-7fac-483b-aaf5-b83d764d0176"
-      (reference "U1") (unit 2) (value "LF412") (footprint "Package_DIP:DIP-8_W10.16mm_LongPads")
+      (reference "U1") (unit 2) (value "LF412") (footprint "Package_DIP:DIP-8_W7.62mm_Socket_LongPads")
     )
     (path "/4d16f993-014c-4d7a-afc5-3442f5282af5"
-      (reference "U1") (unit 3) (value "LF412") (footprint "Package_DIP:DIP-8_W10.16mm_LongPads")
-    )
-  )
+      (reference "U1") (unit 3) (value "LF412") (footprint "Package_DIP:DIP-8_W7.62mm_Socket_LongPads")
+    )
+  )

Commit message: Added test points, changed 2n7000 T0-92 footprint
Parts:
- Q3: footprint Package_TO_SOT_THT:TO-92_Inline -> Package_TO_SOT_THT:TO-92_HandSolder
Changed lines of the file:
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@@
     (title "Peltier PID controller lab electronics ")
     (date "2022-01-06")
-    (rev "1")
+    (rev "2")
     (company "McGill University")
   )
@@
       (effects (font (size 1.27 1.27)) (justify left))
     )
-    (property "Footprint" "Package_TO_SOT_THT:TO-92_Inline" (id 2) (at 137.795 103.505 0)
+    (property "Footprint" "Package_TO_SOT_THT:TO-92_HandSolder" (id 2) (at 137.795 103.505 0)
       (effects (font (size 1.27 1.27) italic) (justify left) hide)
     )
@@
     )
     (path "/8862d4f2-229b-4cfb-89d1-19b80d2e8ad2"
-      (reference "Q3") (unit 1) (value "2N7000") (footprint "Package_TO_SOT_THT:TO-92_Inline")
+      (reference "Q3") (unit 1) (value "2N7000") (footprint "Package_TO_SOT_THT:TO-92_HandSolder")
     )
     (path "/7ce74685-9a6c-4496-92be-75c552d48a24"
